Commit message: deadman

File: description/properties.xacro (robot description, xacro)
@@ -14,3 +14,6 @@
         <color rgba= "0 0 0 1"/>
     </material>
+    <material name="red">
+        <color rgba= "1 0 0 1"/>
+    </material>
 </robot>

File: description/robot.urdf.xacro (robot description, xacro)
@@ -6,3 +6,4 @@
     <xacro:include filename="inertial_macros.xacro"/>
     <xacro:include filename="gazebo_control.xacro"/>
+    <xacro:include filename="lidar.xacro"/>
 </robot>

File: description/robot_core.xacro (robot description, xacro)
@@ -19,5 +19,4 @@
             </geometry>
             <material name="white"/>
-           <!--  <material>Gazebo/White</material>-->
         </visual>
         <collision>
@@ -31,4 +30,7 @@
         </xacro:inertial_box>
     </link>
+    <gazebo reference="chassis">
+        <material>Gazebo/White</material>
+    </gazebo>
     <!-- left wheel joint -->
     <joint name="left_wheel_joint" type="continuous">
@@ -45,5 +47,4 @@
             </geometry>
             <material name="blue"/>
-          <!--   <material>Gazebo/Blue</material> -->
         </visual>
         <collision>
@@ -56,4 +57,7 @@
         </xacro:inertial_cylinder>
     </link>
+    <gazebo reference="left_wheel">
+        <material>Gazebo/Blue</material>
+    </gazebo>
     <!-- right wheel joint -->
     <joint name="right_wheel_joint" type="continuous">
@@ -70,5 +74,4 @@
             </geometry>
             <material name="blue"/>
-            <!-- <material>Gazebo/Blue</material>-->
         </visual>
         <collision>
@@ -81,4 +84,7 @@
         </xacro:inertial_cylinder>
     </link>
+    <gazebo reference="right_wheel">
+        <material>Gazebo/Blue</material>
+    </gazebo>
     <!-- caster wheel joint -->
     <joint name="caster_wheel_joint" type="fixed">
@@ -94,7 +100,4 @@
             </geometry>
             <material name="black"/>
-            <!-- <material>Gazebo/Black</material>
-             <mu1 value = "0.001" />
-            <mu2 value = "0.001" />-->
         </visual>
         <collision>
@@ -107,3 +110,8 @@
         </xacro:inertial_sphere>
     </link>
+    <gazebo reference="caster_wheel">
+        <material>Gazebo/Black</material>
+        <mu1 value = "0.001" />
+        <mu2 value = "0.001" />
+    </gazebo>
 </robot>
