Commit message: Cambios

File: description/robot_core.xacro (robot description, xacro)
@@ -11,4 +11,12 @@
         <origin xyz="-0.1 0 0"/>
     </joint>
+    <!--esta huella es para el perimetro la informacion  este es mi volumen y puedo pasar -->
+    <joint name="base_footprint_joint" type="fixed">
+        <parent link="base_link"/>
+        <child link="base_footprint"/>
+        <origin xyz="0 0 -0.025"/>
+    </joint>
+    <link name="base_footprint">
+    </link>
     <!-- chassis link -->
     <link name="chassis">

Commit message: URDF modelo Ackerman

File: description/robot_core.xacro (robot description, xacro)
@@ -9,5 +9,5 @@
         <parent link="base_link"/>
         <child link="chassis"/>
-        <origin xyz="-0.1 0 0"/>
+        <origin xyz="-0.065 0 0"/>
     </joint>
     <!--esta huella es para el perimetro la informacion  este es mi volumen y puedo pasar -->
@@ -15,5 +15,5 @@
         <parent link="base_link"/>
         <child link="base_footprint"/>
-        <origin xyz="0 0 -0.025"/>
+        <origin xyz="0 0 -0.035"/>
     </joint>
     <link name="base_footprint">
@@ -24,5 +24,5 @@
             <origin xyz="0.15 0 0.075"/>
             <geometry>
-                <box size="0.3 0.3 0.15"/>
+                <box size="0.3 0.2 0.15"/>
             </geometry>
             <material name="white"/>
@@ -45,5 +45,5 @@
         <parent link="base_link"/>
         <child link="left_wheel"/>
-        <origin xyz="0 0.175 0" rpy="-${pi/2} 0 0"/>
+        <origin xyz="0 0.12 0" rpy="-${pi/2} 0 0"/>
         <axis xyz="0 0 1"/>
     </joint>
@@ -52,15 +52,15 @@
         <visual>
             <geometry>
-                <cylinder radius="0.05" length="0.04"/>
-            </geometry>
-            <material name="blue"/>
-        </visual>
-        <collision>
-            <geometry>
-                <cylinder radius="0.05" length="0.04"/>
-            </geometry>
-        </collision>
-        <xacro:inertial_cylinder mass="0.1" length="0.04" radius="0.05">
-            <origin xyz="0 0 0" rpy="0 0 0"/>
+                <cylinder radius="0.035" length="0.04"/>
+            </geometry>
+            <material name="blue"/>
+        </visual>
+        <collision>
+            <geometry>
+                <cylinder radius="0.035" length="0.04"/>
+            </geometry>
+        </collision>
+        <xacro:inertial_cylinder mass="0.1" length="0.04" radius="0.035">
+            <origin xyz="0 0.1 0" rpy="0 0 0"/>
         </xacro:inertial_cylinder>
     </link>
@@ -72,5 +72,5 @@
         <parent link="base_link"/>
         <child link="right_wheel"/>
-        <origin xyz="0 -0.175 0" rpy="${pi/2} 0 0"/>
+        <origin xyz="0 -0.12 0" rpy="${pi/2} 0 0"/>
         <axis xyz="0 0 -1"/>
     </joint>
@@ -79,14 +79,14 @@
         <visual>
             <geometry>
-                <cylinder radius="0.05" length="0.04"/>
-            </geometry>
-            <material name="blue"/>
-        </visual>
-        <collision>
-            <geometry>
-                <cylinder radius="0.05" length="0.04"/>
-            </geometry>
-        </collision>
-        <xacro:inertial_cylinder mass="0.1" length="0.04" radius="0.05">
+                <cylinder radius="0.035" length="0.04"/>
+            </geometry>
+            <material name="blue"/>
+        </visual>
+        <collision>
+            <geometry>
+                <cylinder radius="0.035" length="0.04"/>
+            </geometry>
+        </collision>
+        <xacro:inertial_cylinder mass="0.1" length="0.04" radius="0.035">
             <origin xyz="0 0 0" rpy="0 0 0"/>
         </xacro:inertial_cylinder>
@@ -95,31 +95,113 @@
         <material>Gazebo/Blue</material>
     </gazebo>
-    <!-- caster wheel joint -->
-    <joint name="caster_wheel_joint" type="fixed">
+    <!-- front left wheel steer joint -->
+    <joint name="left_wheel_steer_joint" type="revolute">
+        <limit lower="-1" upper="1" effort="1" velocity="5"/>
         <parent link="chassis"/>
-        <child link="caster_wheel"/>
-        <origin xyz="0.24 0 0"/>
-    </joint>
-    <!-- left wheel link -->
-    <link name="caster_wheel">
-        <visual>
-            <geometry>
-                <sphere radius="0.05"/>
-            </geometry>
-            <material name="black"/>
-        </visual>
-        <collision>
-            <geometry>
-                <sphere radius="0.05"/>
-            </geometry>
-        </collision>
-        <xacro:inertial_sphere mass="0.1" radius="0.05">
-            <origin xyz="0 0 0" rpy="0 0 0"/>
-        </xacro:inertial_sphere>
-    </link>
-    <gazebo reference="caster_wheel">
-        <material>Gazebo/Black</material>
-        <mu1 value = "0.001" />
-        <mu2 value = "0.001" />
+        <child link="left_wheel_steer"/>
+        <origin xyz="0.235 0.12 0" rpy="0 0 0"/>
+        <axis xyz="0 0 1"/>
+    </joint>
+    <!-- front left wheel steer link -->
+    <link name="left_wheel_steer">
+        <visual>
+            <geometry>
+                <cylinder radius="0.001" length="0.001"/>
+            </geometry>
+            <material name="blue"/>
+        </visual>
+        <collision>
+            <geometry>
+                <cylinder radius="0.001" length="0.001"/>
+            </geometry>
+        </collision>
+        <xacro:inertial_cylinder mass="0.001" length="0.001" radius="0.001">
+            <origin xyz="0 0 0" rpy="0 0 0"/>
+        </xacro:inertial_cylinder>
+    </link>
+    <gazebo reference="left_wheel_steer">
+        <material>Gazebo/Blue</material>
+    </gazebo>
+    <!-- front left wheel joint -->
+    <joint name="F_left_wheel_joint" type="continuous">
+        <parent link="left_wheel_steer"/>
+        <child link="F_left_wheel"/>
+        <origin xyz="0 0 0" rpy="-${pi/2} 0 0"/>
+        <axis xyz="0 0 1"/>
+    </joint>
+    <!-- front left wheel link -->
+    <link name="F_left_wheel">
+        <visual>
+            <geometry>
+                <cylinder radius="0.035" length="0.04"/>
+            </geometry>
+            <material name="blue"/>
+        </visual>
+        <collision>
+            <geometry>
+                <cylinder radius="0.035" length="0.04"/>
+            </geometry>
+        </collision>
+        <xacro:inertial_cylinder mass="0.1" length="0.04" radius="0.035">
+            <origin xyz="0 0 0" rpy="0 0 0"/>
+        </xacro:inertial_cylinder>
+    </link>
+    <gazebo reference="F_left_wheel">
+        <material>Gazebo/Blue</material>
+    </gazebo>
+    <!-- front right wheel steer joint -->
+    <joint name="right_wheel_steer_joint" type="revolute">
+        <limit lower="-1" upper="1" effort="1" velocity="5"/>
+        <parent link="chassis"/>
+        <child link="right_wheel_steer"/>
+        <origin xyz="0.235 -0.12 0" rpy="0 0 0"/>
+        <axis xyz="0 0 1"/>
+    </joint>
+    <!-- front left wheel steer link -->
+    <link name="right_wheel_steer">
+        <visual>
+            <geometry>
+                <cylinder radius="0.001" length="0.001"/>
+            </geometry>
+            <material name="blue"/>
+        </visual>
+        <collision>
+            <geometry>
+                <cylinder radius="0.001" length="0.001"/>
+            </geometry>
+        </collision>
+        <xacro:inertial_cylinder mass="0.001" length="0.001" radius="0.001">
+            <origin xyz="0 0 0" rpy="0 0 0"/>
+        </xacro:inertial_cylinder>
+    </link>
+    <gazebo reference="right_wheel_steer">
+        <material>Gazebo/Blue</material>
+    </gazebo>
+    <!-- front right wheel joint -->
+    <joint name="F_right_wheel_joint" type="continuous">
+        <parent link="right_wheel_steer"/>
+        <child link="F_right_wheel"/>
+        <origin xyz="0 0 0" rpy="${pi/2} 0 0"/>
+        <axis xyz="0 0 1"/>
+    </joint>
+    <!-- front right wheel link -->
+    <link name="F_right_wheel">
+        <visual>
+            <geometry>
+                <cylinder radius="0.035" length="0.04"/>
+            </geometry>
+            <material name="blue"/>
+        </visual>
+        <collision>
+            <geometry>
+                <cylinder radius="0.035" length="0.04"/>
+            </geometry>
+        </collision>
+        <xacro:inertial_cylinder mass="0.1" length="0.04" radius="0.035">
+            <origin xyz="0 0 0" rpy="0 0 0"/>
+        </xacro:inertial_cylinder>
+    </link>
+    <gazebo reference="F_right_wheel">
+        <material>Gazebo/Blue</material>
     </gazebo>
 </robot>
