Commit message: COMMIT ADELANTO

File: description/robot.urdf.xacro (robot description, xacro)
@@ -2,6 +2,7 @@
 <robot xmlns:xacro="http://www.ros.org/wiki/xacro"  name="robot">
     <!-- Example link -->
+    <xacro:include filename="properties.xacro"/>
     <xacro:include filename="robot_core.xacro"/>
-        <!-- Example link -->
-    <link name="base_link"></link>
+    <xacro:include filename="inertial_macros.xacro"/>
+    <xacro:include filename="gazebo_control.xacro"/>
 </robot>

Commit message: Inital branch commit

File: description/robot.urdf.xacro (robot description, xacro)
@@ -5,5 +5,6 @@
     <xacro:include filename="robot_core.xacro"/>
     <xacro:include filename="inertial_macros.xacro"/>
-    <xacro:include filename="gazebo_control.xacro"/>
+    <!-- <xacro:include filename="gazebo_control.xacro"/> -->
     <xacro:include filename="lidar.xacro"/>
+    <xacro:include filename="ros2_control.xacro"/>
 </robot>

File: description/robot_core.xacro (robot description, xacro)
@@ -58,5 +58,6 @@
         <collision>
             <geometry>
-                <cylinder radius="0.05" length="0.04"/>
+                <!-- <cylinder radius="0.05" length="0.04"/> -->
+                <sphere radius="0.05"/>
             </geometry>
         </collision>
@@ -85,5 +86,6 @@
         <collision>
             <geometry>
-                <cylinder radius="0.05" length="0.04"/>
+                <!-- <cylinder radius="0.05" length="0.04"/> -->
+                <sphere radius="0.05"/>
             </geometry>
         </collision>
