Commit message: 8/09/2023 no esta el ackerman completo, esto fue justo antes del parcial

File: description/lidar.xacro (robot description, xacro)
@@ -28,5 +28,5 @@
         <sensor name="laser" type="ray">
             <pose>0 0 0 0 0 0</pose>
-            <visualize>true</visualize>
+            <visualize>true</visualize> <!--aqui se le dice si quiero ver o no los rayos-->
             <update_rate>10</update_rate>
             <ray>

File: description/robot.urdf.xacro (robot description, xacro)
@@ -5,5 +5,6 @@
     <xacro:include filename="robot_core.xacro"/>
     <xacro:include filename="inertial_macros.xacro"/>
-    <xacro:include filename="gazebo_control.xacro"/>
+    <!--<xacro:include filename="gazebo_control.xacro"/>-->
     <xacro:include filename="lidar.xacro"/>
+    <xacro:include filename="ros2_control.xacro"/>
 </robot>

File: description/robot_core.xacro (robot description, xacro)
@@ -31,5 +31,5 @@
             <origin xyz="0.15 0 0.075"/>
             <geometry>
-                <box size="0.3 0.3 0.15"/>
+                <box size="0.3 0.2 0.15"/>
             </geometry>
         </collision>
@@ -58,5 +58,5 @@
         <collision>
             <geometry>
-                <cylinder radius="0.035" length="0.04"/>
+                <sphere radius="0.035"/>
             </geometry>
         </collision>
@@ -85,5 +85,5 @@
         <collision>
             <geometry>
-                <cylinder radius="0.035" length="0.04"/>
+                <sphere radius="0.035"/>
             </geometry>
         </collision>
@@ -113,5 +113,5 @@
         <collision>
             <geometry>
-                <cylinder radius="0.001" length="0.001"/>
+                <sphere radius="0.001"/>
             </geometry>
         </collision>
@@ -140,5 +140,5 @@
         <collision>
             <geometry>
-                <cylinder radius="0.035" length="0.04"/>
+                <sphere radius="0.035"/>
             </geometry>
         </collision>
@@ -168,5 +168,5 @@
         <collision>
             <geometry>
-                <cylinder radius="0.001" length="0.001"/>
+                <sphere radius="0.001"/>
             </geometry>
         </collision>
@@ -195,5 +195,5 @@
         <collision>
             <geometry>
-                <cylinder radius="0.035" length="0.04"/>
+                <sphere radius="0.035"/>
             </geometry>
         </collision>
