Commit message: Ackerman no esta completo, esto es antes del parcial

File: description/gazebo_control.xacro (robot description, xacro)
@@ -1,21 +1,29 @@
 <?xml version="1.0"?>
 <robot xmlns:xacro="http://www.ros.org/wiki/xacro" >
-    <!-- Example link -->
     <gazebo>
-        <plugin name="diff_drive" filename="libgazebo_ros_diff_drive.so">
-            <!-- wheels information -->
-            <left_joint>left_wheel_joint</left_joint>
-            <right_joint>right_wheel_joint</right_joint>
-            <wheel_separation>0.35</wheel_separation>
-            <wheel_diameter>0.1</wheel_diameter>
-            <!-- limits -->
-            <max_wheel_torque>200</max_wheel_torque>
-            <max_wheel_acceleration>10.0</max_wheel_acceleration>
-            <!-- outputs -->
-            <odometry_frame>odom</odometry_frame>
-            <robot_base_frame>base_link</robot_base_frame>
-            <publish_odom>true</publish_odom>
-            <publish_odom_tf>true</publish_odom_tf>
-            <publish_wheel_tf>true</publish_wheel_tf>
+        <plugin name="gazebo_ros_ackermann_drive" filename="libgazebo_ros_ackermann_drive.so">
+            <ros>
+                <namespace>demo</namespace>
+                <argument>cmd_vel:=cmd_demo</argument>
+                <argument>odom:=odom_demo</argument>
+                <argument>distance:=distance_demo</argument>
+            </ros>
+            <update_rate>100.0</update_rate>
+            <!-- wheels -->
+            <front_left_joint>front_left_wheel_joint</front_left_joint>
+            <front_right_joint>front_right_wheel_joint</front_right_joint>
+            <rear_left_joint>rear_left_wheel_joint</rear_left_joint>
+            <rear_right_joint>rear_right_wheel_joint</rear_right_joint>
+            <left_steering_joint>front_left_steer_joint</left_steering_joint>
+            <right_steering_joint>front_right_steer_joint</right_steering_joint>
+            <steering_wheel_joint>steering_joint</steering_wheel_joint>
+            <!-- Max absolute steer angle for tyre in radians-->
+            <max_steer>0.6458</max_steer>
+            <!-- Max absolute steering angle of steering wheel -->
+            <max_steering_angle>7.85</max_steering_angle>
+            <!-- Max absolute linear speed in m/s -->
+            <max_speed>20</max_speed>
+            <odometry_frame>odom_demo</odometry_frame>
+            <robot_base_frame>chassis</robot_base_frame>
         </plugin>
     </gazebo>

File: description/lidar.xacro (robot description, xacro)
@@ -33,8 +33,8 @@
                 <scan>
                     <horizontal>
-                        <samples>360</samples>
+                        <samples>180</samples>
                         <resolution>1</resolution>
-                        <min_angle>-3.14</min_angle>
-                        <max_angle>3.14</max_angle>
+                        <min_angle>-1.57</min_angle>
+                        <max_angle>1.57</max_angle>
                     </horizontal>
                 </scan>

File: description/robot.urdf.xacro (robot description, xacro)
@@ -3,7 +3,8 @@
     <!-- Example link -->
     <xacro:include filename="properties.xacro"/>
-    <xacro:include filename="robot_core.xacro"/>
+    <!-- <xacro:include filename="robot_core.xacro"/> -->
+    <xacro:include filename="robot_core_dif.xacro"/>
     <xacro:include filename="inertial_macros.xacro"/>
-    <!--<xacro:include filename="gazebo_control.xacro"/>-->
+    <!-- <xacro:include filename="gazebo_control.xacro"/> -->
     <xacro:include filename="lidar.xacro"/>
     <xacro:include filename="ros2_control.xacro"/>

File: description/robot_core.xacro (robot description, xacro)
@@ -95,10 +95,38 @@
         <material>Gazebo/Blue</material>
     </gazebo>
+    <!-- steering joint -->
+    <joint name="steering_joint" type="revolute">
+        <limit lower="-1" upper="1" effort="1" velocity="5"/>
+        <parent link="base_link"/>
+        <child link="steering_wheel"/>
+        <origin xyz="0.17 0 0" rpy="0 0 0"/>
+        <axis xyz="0 0 1"/>
+    </joint>
+    <!-- steering link -->
+    <link name="steering_wheel">
+        <visual>
+            <geometry>
+                <cylinder radius="0.001" length="0.001"/>
+            </geometry>
+            <material name="blue"/>
+        </visual>
+        <collision>
+            <geometry>
+                <sphere radius="0.001"/>
+            </geometry>
+        </collision>
+        <xacro:inertial_cylinder mass="0.001" length="0.001" radius="0.001">
+            <origin xyz="0 0 0" rpy="0 0 0"/>
+        </xacro:inertial_cylinder>
+    </link>
+    <gazebo reference="steering_wheel">
+        <material>Gazebo/Blue</material>
+    </gazebo>
     <!-- front left wheel steer joint -->
-    <joint name="left_wheel_steer_joint" type="revolute">
+    <joint name="front_left_steer_joint" type="revolute">
         <limit lower="-1" upper="1" effort="1" velocity="5"/>
-        <parent link="chassis"/>
+        <parent link="base_link"/>
         <child link="left_wheel_steer"/>
-        <origin xyz="0.235 0.12 0" rpy="0 0 0"/>
+        <origin xyz="0.17 0.12 0" rpy="0 0 0"/>
         <axis xyz="0 0 1"/>
     </joint>
@@ -124,5 +152,5 @@
     </gazebo>
     <!-- front left wheel joint -->
-    <joint name="F_left_wheel_joint" type="continuous">
+    <joint name="front_left_wheel_joint" type="continuous">
         <parent link="left_wheel_steer"/>
         <child link="F_left_wheel"/>
@@ -151,9 +179,9 @@
     </gazebo>
     <!-- front right wheel steer joint -->
-    <joint name="right_wheel_steer_joint" type="revolute">
+    <joint name="front_right_steer_joint" type="revolute">
         <limit lower="-1" upper="1" effort="1" velocity="5"/>
-        <parent link="chassis"/>
+        <parent link="base_link"/>
         <child link="right_wheel_steer"/>
-        <origin xyz="0.235 -0.12 0" rpy="0 0 0"/>
+        <origin xyz="0.17 -0.12 0" rpy="0 0 0"/>
         <axis xyz="0 0 1"/>
     </joint>
@@ -178,6 +206,6 @@
         <material>Gazebo/Blue</material>
     </gazebo>
-    <!-- front right wheel joint -->
-    <joint name="F_right_wheel_joint" type="continuous">
+    <!--front right wheel joint -->
+    <joint name="front_right_wheel_joint" type="continuous">
         <parent link="right_wheel_steer"/>
         <child link="F_right_wheel"/>
